File: Resources/h bridge dev board/h_bridge_dev_board.sch (EAGLE design)
At the start: 26 parts, among them IC1 74LS08N, IC2 74LS08N, IC3 74LS08N, IC4 7404N, IC5 74LS595N, IC6 74158N

Commit message: minor update in schematic
Parts:
- removed X3: (no value), con-wago-500:W237-4
- added OUT_A_B, OUT_C_D: (no value), con-wago-500:W237-102
- added POWER: (no value), con-wago-500:W237-4
- added RN2: (no value), resistor-sil:G05R
- added SW1: (no value), special:SW_DIP-4
- renumbered X1 to CHN_A_B, X2 to CHN_C_D
Connections:
- removed net N$10: IC6A.4Y
- removed net N$24: IC1A.O
- removed net N$25: IC1B.O
- removed net N$26: IC1C.O
- removed net N$27: IC1D.O
- removed net N$28: IC2A.O
- removed net N$29: IC2B.O
- removed net N$3: D5.C, D6.C, U$5.COLLECTOR, U$6.COLLECTOR
- removed net N$30: IC2C.O
- removed net N$31: IC2D.O
- removed net N$4: IC6A.1Y
- removed net N$5: IC6A.2Y
- removed net N$6: D7.A, D8.A, U$7.EMITTER
- removed net N$61: U$1.BASE
- removed net N$7: D3.A, D4.A, U$2.EMITTER, U$4.EMITTER
- removed net N$8: D1.C, D2.C, U$1.COLLECTOR
- removed net N$9: IC6A.3Y
- new net 5V: POWER-4.KL
- new net AH1: IC1A.O, U$1.BASE
- new net AH2: IC2A.O, U$5.BASE
- new net AL1: IC1B.O, U$2.BASE
- new net AL2: IC2B.O, U$7.BASE
- new net BH1: IC1C.O, U$3.BASE
- new net BH2: IC2C.O, U$6.BASE
- new net BL1: IC1D.O, U$4.BASE
- new net BL2: IC2D.O, U$8.BASE
- new net CCP1: PCB1.D9
- new net CCP2: PCB1.D10
- new net CHIP_ENABLE: PCB1.D7, RN2.5, SW1.5
- new net DIR: PCB1.D3
- new net GND: D3.A, D4.A, D7.A, D8.A, PCB1.GND., POWER-2.KL, POWER-3.KL, RN2.1, U$2.EMITTER, U$4.EMITTER, U$7.EMITTER
- new net MS0: PCB1.D4, RN2.2, SW1.8
- new net MS1: PCB1.D5, RN2.3, SW1.7
- new net MS2: PCB1.D6, RN2.4, SW1.6
- new net SENSE01: PCB1.A0
- new net SENSE02: PCB1.A1
- new net STEP: PCB1.D2
- new net VCC: D1.C, D2.C, D5.C, D6.C, POWER-1.KL, U$1.COLLECTOR, U$5.COLLECTOR, U$6.COLLECTOR
- net +5V: now also PCB1.VIN, SW1.1, SW1.2, SW1.3, SW1.4
- net DS: now also PCB1.A5
- net MR: now also PCB1.A4
- net OE: now also PCB1.D12
- net OUT_A: now also OUT_A_B-1.KL; no longer X3-1.KL
- net OUT_B: now also OUT_A_B-2.KL; no longer X3-2.KL
- net OUT_C: now also OUT_C_D-1.KL; no longer X3-3.KL
- net OUT_D: now also OUT_C_D-2.KL; no longer X3-4.KL
- net SH_CP: now also PCB1.A2
- net ST_CP: now also PCB1.A3
- net Y1: now also IC6A.1Y
- net Y2: now also IC6A.2Y
- net Y3: now also IC6A.3Y
- net Y4: now also IC6A.4Y

Commit message: dev board schematic nearly complete
Parts:
- removed U$1, U$2, U$3, U$4, U$5, U$6, U$7, U$8: TIP35_STYLE3, tip35_style3:TIP35_STYLE3
- added AH, AL, BH, BL, CH, CL, DH, DL: TIP35_STYLE3, tip35_style3:TIP35_STYLE3
- added CAP_AH, CAP_AL, CAP_BH, CAP_BL, CAP_CH, CAP_CL, CAP_DH, CAP_DL, DB_AH, DB_AL, DB_BH, DB_BL, DB_CH, DB_CL, DB_DH, DB_DL, DF_AH, DF_AL, DF_BH, DF_BL, DF_CH, DF_CL, DF_DH, DF_DL, DR_AH, DR_AL, DR_BH, DR_BL, DR_CH, DR_CL, DR_DH, DR_DL, RES_BASE_AH, RES_BASE_AL, RES_BASE_BH, RES_BASE_BL, RES_BASE_CH, RES_BASE_CL, RES_BASE_DH, RES_BASE_DL: J30MM, jumper:J30MM
- added IC7: LM358N, linear:LM358N
- added INTERFACE: (no value), pinhead:PINHD-1X7/90
- added J25, J26, J27, J28: J50MM, jumper:J50MM
- RN2: value (none) -> 103G
Connections:
- removed net AH1: IC1A.O, U$1.BASE
- removed net AH2: IC2A.O, U$5.BASE
- removed net AL1: IC1B.O, U$2.BASE
- removed net AL2: IC2B.O, U$7.BASE
- removed net BH1: IC1C.O, U$3.BASE
- removed net BH2: IC2C.O, U$6.BASE
- removed net BL1: IC1D.O, U$4.BASE
- removed net BL2: IC2D.O, U$8.BASE
- removed net N$12: IC6A.1A
- removed net N$14: IC6A.2A
- removed net N$15: IC6A.3A
- removed net N$16: IC6A.4A
- removed net N$17: IC6A.!A!/B
- removed net N$18: IC6A.G
- new net AH: AH.BASE, DB_AH.2, DR_AH.2
- new net AL: AL.BASE, DB_AL.2, DR_AL.2
- new net BAKER_CLAMP_AH: IC1A.O, RES_BASE_AH.1
- new net BAKER_CLAMP_AL: IC1B.O, RES_BASE_AL.1
- new net BAKER_CLAMP_BH: IC1C.O, RES_BASE_BH.2
- new net BAKER_CLAMP_BL: IC1D.O, RES_BASE_BL.2
- new net BAKER_CLAMP_CH: IC2A.O, RES_BASE_CH.2
- new net BAKER_CLAMP_CL: IC2B.O, RES_BASE_CL.1
- new net BAKER_CLAMP_DH: IC2C.O, RES_BASE_DH.2
- new net BAKER_CLAMP_DL: IC2D.O, RES_BASE_DL.2
- new net BH: BH.BASE, DB_BH.2, DR_BH.2
- new net BL: BL.BASE, DB_BL.2, DR_BL.2
- new net CH: CH.BASE, DB_CH.2, DR_CH.2
- new net CL: CL.BASE, DB_CL.2, DR_CL.2
- new net DH: DB_DH.2, DH.BASE, DR_DH.2
- new net DL: DB_DL.2, DL.BASE, DR_DL.2
- new net N$10: CAP_AL.1, RES_BASE_AL.2
- new net N$19: CAP_CL.2, DB_CL.1, DF_CL.1, DR_CL.1
- new net N$2: IC1P.GND, IC2P.GND, IC3P.GND, IC4P.GND, IC5P.GND, IC6P.GND
- new net N$20: CAP_AH.2, DB_AH.1, DF_AH.1, DR_AH.1
- new net N$21: CAP_BH.1, DB_BH.1, DF_BH.1, DR_BH.1
- new net N$22: CAP_CH.1, RES_BASE_CH.1
- new net N$23: CAP_CL.1, RES_BASE_CL.2
- new net N$24: CAP_BH.2, RES_BASE_BH.1
- new net N$26: CAP_BL.2, RES_BASE_BL.1
- new net N$28: CAP_DH.2, RES_BASE_DH.1
- new net N$29: CAP_DL.2, RES_BASE_DL.1
- new net N$4: CAP_AL.2, DB_AL.1, DF_AL.1, DR_AL.1
- new net N$5: CAP_CH.2, DB_CH.1, DF_CH.1, DR_CH.1
- new net N$6: CAP_BL.1, DB_BL.1, DF_BL.1, DR_BL.1
- new net N$7: DB_DL.1, DF_DL.1, DR_DL.1
- new net N$8: CAP_DH.1, DB_DH.1, DF_DH.1, DR_DH.1
- new net N$9: CAP_AH.1, RES_BASE_AH.2
- new net R_SENSE_A_B: AL.EMITTER, BL.EMITTER, D3.A, D4.A, J27.2, J28.1
- new net R_SENSE_C_D: CL.EMITTER, D7.A, D8.A, DL.EMITTER, J25.2, J26.1
- net +5V: now also IC1P.VCC, IC2P.VCC, IC3P.VCC, IC4P.VCC, IC5P.VCC, IC6P.VCC
- net CCP1: now also IC6A.1A, IC6A.2A
- net CCP2: now also IC6A.3A, IC6A.4A
- net CHIP_ENABLE: now also INTERFACE.5
- net DIR: now also INTERFACE.6
- net ENABLE_C_D: now also IC2A.I1, IC2B.I1
- net GND: now also INTERFACE.4, J25.1, J26.2, J27.1, J28.2; no longer D3.A, D4.A, D7.A, D8.A, U$2.EMITTER, U$4.EMITTER, U$7.EMITTER
- net MS0: now also INTERFACE.3
- net MS1: now also INTERFACE.2
- net MS2: now also INTERFACE.1
- net OUT_A: now also AH.EMITTER, AL.COLLECTOR, DF_AL.2; no longer U$1.EMITTER
- net OUT_B: now also BH.EMITTER, BL.COLLECTOR, DF_BL.2; no longer U$3.EMITTER, U$4.COLLECTOR
- net OUT_C: now also CH.EMITTER, CL.COLLECTOR, DF_CL.2; no longer U$5.EMITTER, U$7.COLLECTOR
- net OUT_D: now also DF_DL.2, DH.EMITTER, DL.COLLECTOR; no longer U$6.EMITTER, U$8.COLLECTOR
- net SELECT: now also IC6A.!A!/B
- net STEP: now also INTERFACE.7
- net STROBE: now also IC6A.G
- net VCC: now also AH.COLLECTOR, BH.COLLECTOR, CH.COLLECTOR, DF_AH.2, DF_BH.2, DF_CH.2, DF_DH.2, DH.COLLECTOR; no longer U$1.COLLECTOR, U$5.COLLECTOR, U$6.COLLECTOR
Other:
- moved on the sheet: CHN_A_B-1, CHN_A_B-2, CHN_A_B-3, CHN_C_D-1, CHN_C_D-2, CHN_C_D-3, D1, D2, D3, D4, D5, D6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

Commit message: ADC code working. dev board schematic needs final check
Parts:
- added 6.8V: 1N4738, zener_1n4736A:1N4738
- added C1, C2: 100uF 50v, resistor:CPOL-USE5-13
- added R1: 330 ohm 1w, resistor:R-US_0207/15
- added R_F_AB, R_F_CD, R_G_AB, R_G_CD: J10MM, jumper:J10MM
- added SENSE: (no value), con-wago-500:W237-102
Connections:
- new net +6.5V: 6.8V.C, IC7P.V+, R1.2
- new net N$16: IC7B.-IN, R_F_CD.1, R_G_CD.2
- new net N$18: IC7A.-IN, R_F_AB.1, R_G_AB.2
- net GND: now also 6.8V.A, C1.-, C2.-, IC7P.V-, R_G_AB.1, R_G_CD.1
- net N$7: now also CAP_DL.1
- net R_SENSE_A_B: now also IC7A.+IN
- net R_SENSE_C_D: now also IC7B.+IN
- net SENSE01: now also IC7A.OUT, R_F_AB.2, SENSE-1.KL
- net SENSE02: now also IC7B.OUT, R_F_CD.2, SENSE-2.KL
- net VCC: now also C1.+, C2.+, R1.1
Other:
- moved on the sheet: IC7A, IC7B

Commit message: minor change
Connections:
- removed net N$2: IC1P.GND, IC2P.GND, IC3P.GND, IC4P.GND, IC5P.GND, IC6P.GND
- net GND: now also IC1P.GND, IC2P.GND, IC3P.GND, IC4P.GND, IC5P.GND, IC6P.GND
Changed lines of the file:
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@@
 <wire x1="160.02" y1="-160.02" x2="160.02" y2="-167.64" width="0.1524" layer="91"/>
+</segment>
+<segment>
+<pinref part="IC6" gate="P" pin="GND"/>
+<pinref part="IC5" gate="P" pin="GND"/>
+<wire x1="-325.12" y1="15.24" x2="-325.12" y2="12.7" width="0.1524" layer="91"/>
+<pinref part="IC3" gate="P" pin="GND"/>
+<wire x1="-325.12" y1="12.7" x2="-325.12" y2="10.16" width="0.1524" layer="91"/>
+<wire x1="-325.12" y1="10.16" x2="-325.12" y2="5.08" width="0.1524" layer="91"/>
+<junction x="-325.12" y="10.16"/>
+<pinref part="IC4" gate="P" pin="GND"/>
+<wire x1="-325.12" y1="5.08" x2="-325.12" y2="0" width="0.1524" layer="91"/>
+<junction x="-325.12" y="5.08"/>
+<pinref part="IC1" gate="P" pin="GND"/>
+<wire x1="-325.12" y1="0" x2="-325.12" y2="-5.08" width="0.1524" layer="91"/>
+<junction x="-325.12" y="0"/>
+<pinref part="IC2" gate="P" pin="GND"/>
+<wire x1="-325.12" y1="-5.08" x2="-325.12" y2="-12.7" width="0.1524" layer="91"/>
+<junction x="-325.12" y="-5.08"/>
+<pinref part="GND6" gate="1" pin="GND"/>
+<wire x1="-325.12" y1="12.7" x2="-314.96" y2="12.7" width="0.1524" layer="91"/>
+<wire x1="-314.96" y1="12.7" x2="-314.96" y2="10.16" width="0.1524" layer="91"/>
+<junction x="-325.12" y="12.7"/>
 </segment>
 </net>
@@
 </segment>
 </net>
-<net name="N$2" class="0">
-<segment>
-<pinref part="IC6" gate="P" pin="GND"/>
-<pinref part="IC5" gate="P" pin="GND"/>
-<wire x1="-325.12" y1="15.24" x2="-325.12" y2="10.16" width="0.1524" layer="91"/>
-<pinref part="IC3" gate="P" pin="GND"/>
-<wire x1="-325.12" y1="10.16" x2="-325.12" y2="5.08" width="0.1524" layer="91"/>
-<junction x="-325.12" y="10.16"/>
-<pinref part="IC4" gate="P" pin="GND"/>
-<wire x1="-325.12" y1="5.08" x2="-325.12" y2="0" width="0.1524" layer="91"/>
-<junction x="-325.12" y="5.08"/>
-<pinref part="IC1" gate="P" pin="GND"/>
-<wire x1="-325.12" y1="0" x2="-325.12" y2="-5.08" width="0.1524" layer="91"/>
-<junction x="-325.12" y="0"/>
-<pinref part="IC2" gate="P" pin="GND"/>
-<wire x1="-325.12" y1="-5.08" x2="-325.12" y2="-12.7" width="0.1524" layer="91"/>
-<junction x="-325.12" y="-5.08"/>
-</segment>
-</net>

Commit message: Major schematic change. swapped few pins. code needs update
Parts:
- added J1, J2, J3, J4: J50MM, jumper:J50MM
- added R2: 3k, resistor:R-US_0207/12
- added R3: 10k, resistor:R-US_0207/12
- added SHIFT_REG: (no value), con-lstb:MA08-2
- added SV2, SV3, SV4, SV5: (no value), con-lsta:FE08-1
- added SV6: (no value), con-lstb:MA03-2
- added SW_DPDT: (no value), switch:A68-A31
- added VREF: 1k, pot:TRIM_US-B25U
- INTERFACE: device pinhead:PINHD-1X7/90 -> con-lstb:MA07-2
Connections:
- new net 3V3: PCB1.3V3, SV4.7
- new net A0: PCB1.A0, SV4.5, SV6.6
- new net A1: PCB1.A1, SV4.4, SV6.4
- new net A2: PCB1.A2, SV4.3, SV6.2
- new net A3: PCB1.A3, SV4.2
- new net A4: PCB1.A4, SHIFT_REG.1, SV4.1
- new net A5: PCB1.A5, SHIFT_REG.3, SV5.8
- new net A6: PCB1.A6, SHIFT_REG.5, SV5.7
- new net A7: PCB1.A7, SV5.6
- new net D10: PCB1.D10, SHIFT_REG.11, SV2.3
- new net D11: PCB1.D11, SHIFT_REG.9, SV2.2
- new net D12: PCB1.D12, SHIFT_REG.7, SV2.1
- new net D13: PCB1.D13, SV4.8
- new net D2: INTERFACE.10, PCB1.D2, SV3.3
- new net D3: INTERFACE.12, PCB1.D3, SV3.2
- new net D4: INTERFACE.2, PCB1.D4, SV3.1
- new net D5: INTERFACE.4, PCB1.D5, SV2.8
- new net D6: INTERFACE.6, PCB1.D6, SV2.7
- new net D7: INTERFACE.8, PCB1.D7, SV2.6
- new net D8: PCB1.D8, SV2.5
- new net D9: PCB1.D9, SHIFT_REG.13, SV2.4
- new net N$2: R2.1, R3.2, VREF.E
- new net N$31: SHIFT_REG.15
- new net N$40: SV3.8
- new net N$56: SV5.1
- new net REF: PCB1.REF, SV4.6
- new net RST: PCB1.RST, PCB1.RST., SV3.5, SV5.4
- new net RX1: PCB1.RX0, SV3.6
- new net TEMP: SHIFT_REG.16
- new net TX1: PCB1.TX1, SV3.7
- new net VIN: PCB1.VIN, SV5.2, SW_DPDTA.S
- new net VREF: SV6.1, VREF.S
- new net V_LOGIC: POWER-4.KL, SW_DPDTB.S
- net +5V: now also R2.2, SW_DPDTA.P, SW_DPDTB.P; no longer PCB1.VIN
- net 5V: now also PCB1.5V, SV5.5, SW_DPDTA.O; no longer POWER-4.KL
- net CCP1: now also SHIFT_REG.14; no longer PCB1.D9
- net CCP2: now also SHIFT_REG.12; no longer PCB1.D10
- net CHIP_ENABLE: now also INTERFACE.7; no longer INTERFACE.5, PCB1.D7
- net DIR: now also INTERFACE.11; no longer INTERFACE.6, PCB1.D3
- net DS: now also SHIFT_REG.6; no longer PCB1.A5
- net GND: now also INTERFACE.13, INTERFACE.14, J1.1, J2.2, J3.1, J4.2, PCB1.GND, R3.1, SV3.4, SV5.3, VREF.A; no longer INTERFACE.4
- net MR: now also SHIFT_REG.10; no longer PCB1.A4
- net MS0: now also INTERFACE.1; no longer INTERFACE.3, PCB1.D4
- net MS1: now also INTERFACE.3; no longer INTERFACE.2, PCB1.D5
- net MS2: now also INTERFACE.5; no longer INTERFACE.1, PCB1.D6
- net OE: now also SHIFT_REG.8; no longer PCB1.D12
- net R_SENSE_A_B: now also J1.2, J2.1
- net R_SENSE_C_D: now also J3.2, J4.1
- net SENSE01: now also SV6.5; no longer PCB1.A0
- net SENSE02: now also SV6.3; no longer PCB1.A1
- net SH_CP: now also SHIFT_REG.2; no longer PCB1.A2
- net STEP: now also INTERFACE.9; no longer INTERFACE.7, PCB1.D2
- net ST_CP: now also SHIFT_REG.4; no longer PCB1.A3

Commit message: minor schematic update
Parts:
- R2: value 3k -> 3.3k
Other:
- note added: "+5V USB +5v Power Supply"
- note added: "+5v Power Supply"
- note added: "K"
Changed lines of the file:
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@@
 <part name="SV5" library="con-lsta" deviceset="FE08-1" device=""/>
 <part name="SV6" library="con-lstb" deviceset="MA03-2" device=""/>
-<part name="R2" library="resistor" deviceset="R-US_" device="0207/12" value="3k"/>
+<part name="R2" library="resistor" deviceset="R-US_" device="0207/12" value="3.3k"/>
 <part name="R3" library="resistor" deviceset="R-US_" device="0207/12" value="10k"/>
 <part name="P+5" library="supply1" deviceset="+5V" device=""/>
@@
 <sheet>
 <plain>
+<text x="-172.72" y="-152.4" size="1.778" layer="112" rot="R90">+5V USB
++5v Power Supply</text>
+<text x="48.26" y="-53.34" size="1.778" layer="112">K</text>
+<text x="60.96" y="-43.18" size="1.778" layer="112">K</text>
+<text x="60.96" y="-33.02" size="1.778" layer="112">K</text>
+<text x="45.72" y="17.78" size="1.778" layer="112">K</text>
+<text x="58.42" y="30.48" size="1.778" layer="112">K</text>
+<text x="55.88" y="43.18" size="1.778" layer="112">K</text>
+<text x="45.72" y="58.42" size="1.778" layer="112">K</text>
+<text x="58.42" y="73.66" size="1.778" layer="112">K</text>
+<text x="55.88" y="83.82" size="1.778" layer="112">K</text>
+<text x="60.96" y="-101.6" size="1.778" layer="112">K</text>
+<text x="63.5" y="-109.22" size="1.778" layer="112">K</text>
+<text x="50.8" y="-119.38" size="1.778" layer="112">K</text>
+<text x="254" y="-121.92" size="1.778" layer="112">K</text>
+<text x="243.84" y="-111.76" size="1.778" layer="112">K</text>
+<text x="243.84" y="-101.6" size="1.778" layer="112">K</text>
+<text x="251.46" y="-50.8" size="1.778" layer="112">K</text>
+<text x="241.3" y="-38.1" size="1.778" layer="112">K</text>
+<text x="241.3" y="-30.48" size="1.778" layer="112">K</text>
+<text x="-91.44" y="81.28" size="1.778" layer="112">+5v Power Supply</text>
 </plain>
 <instances>
@@
 </schematic>
 </drawing>
+<compatibility>
+<note version="6.3" minversion="6.2.2" severity="warning">
+Since Version 6.2.2 text objects can contain more than one line,
+which will not be processed correctly with this version.
+</note>
+</compatibility>
 </eagle>

Commit message: added opto coupler in schematic
Parts:
- added OK1, OK2, OK3, OK4, OK5, OK6, OK7, OK8: PC817, optocoupler:PC817
- added R10, R11, R4, R5, R6, R7, R8, R9: 220, resistor:R-US_0207/10
Connections:
- new net N$12: OK1.A, R4.2
- new net N$14: OK2.A, R5.2
- new net N$15: OK3.A, R6.2
- new net N$17: OK4.A, R7.2
- new net N$27: OK8.A, R11.1
- new net N$30: OK7.A, R10.1
- new net N$32: OK6.A, R9.1
- new net N$33: OK5.A, R8.1
- new net N$34: OK8.EMIT, RES_BASE_DL.2
- new net N$35: OK5.EMIT, RES_BASE_BH.2
- new net N$36: OK6.EMIT, RES_BASE_BL.2
- new net N$37: OK7.EMIT, RES_BASE_DH.2
- new net N$38: OK4.EMIT, RES_BASE_CL.1
- new net N$39: OK3.EMIT, RES_BASE_CH.2
- new net N$42: OK2.EMIT, RES_BASE_AL.1
- new net N$43: OK1.EMIT, RES_BASE_AH.1
- net +5V: now also OK1.COL, OK2.COL, OK3.COL, OK4.COL, OK5.COL, OK6.COL, OK7.COL, OK8.COL
- net BAKER_CLAMP_AH: now also R4.1; no longer RES_BASE_AH.1
- net BAKER_CLAMP_AL: now also R5.1; no longer RES_BASE_AL.1
- net BAKER_CLAMP_BH: now also R8.2; no longer RES_BASE_BH.2
- net BAKER_CLAMP_BL: now also R9.2; no longer RES_BASE_BL.2
- net BAKER_CLAMP_CH: now also R6.1; no longer RES_BASE_CH.2
- net BAKER_CLAMP_CL: now also R7.1; no longer RES_BASE_CL.1
- net BAKER_CLAMP_DH: now also R10.2; no longer RES_BASE_DH.2
- net BAKER_CLAMP_DL: now also R11.2; no longer RES_BASE_DL.2
- net GND: now also OK1.C, OK2.C, OK3.C, OK4.C, OK5.C, OK6.C, OK7.C, OK8.C
Other:
- moved on the sheet: AH, AL, BH, BL, C1, C2, CAP_AH, CAP_AL, CAP_BH, CAP_BL, CAP_CH, CAP_CL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
