File: Resources/h bridge dev board/h_bridge_dev_board.sch (EAGLE design)
At the start: 115 parts, among them IC1 74LS08N, IC2 74LS08N, IC3 74LS08N, IC4 7404N, IC5 74LS595N, IC6 74158N, IC7 LM358N, J1 J50MM, J2 J50MM, J25 J50MM, J26 J50MM, J27 J50MM, J28 J50MM, J3 J50MM, J4 J50MM

Commit message: reduced jumper size in schematic
Parts:
- removed 6.8V: 1N4738, zener_1n4736A:1N4738
- removed R1: 330 ohm 1w, resistor:R-US_0207/15
- CAP_AH, CAP_AL, CAP_BH, CAP_BL, CAP_CH, CAP_CL, CAP_DH, CAP_DL, DB_AH, DB_AL, DB_BH, DB_BL, DB_CH, DB_CL, DB_DH, DB_DL, DF_AH, DF_AL, DF_BH, DF_BL, DF_CH, DF_CL, DF_DH, DF_DL, DR_AH, DR_AL, DR_BH, DR_BL, DR_CH, DR_CL, DR_DH, DR_DL, RES_BASE_AH, RES_BASE_AL, RES_BASE_BH, RES_BASE_BL, RES_BASE_CH, RES_BASE_CL, RES_BASE_DH, RES_BASE_DL: value J30MM -> J15MM; device jumper:J30MM -> jumper:J15MM
Connections:
- removed net +6.5V: 6.8V.C, IC7P.V+, R1.2
- net +5V: now also IC7P.V+
- net GND: no longer 6.8V.A
- net VCC: no longer R1.1
Changed lines of the file:
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@@
 <part name="P+3" library="supply1" deviceset="+5V" device=""/>
 <part name="GND5" library="supply1" deviceset="GND" device=""/>
-<part name="DB_AH" library="jumper" deviceset="J" device="30MM"/>
-<part name="DF_AH" library="jumper" deviceset="J" device="30MM"/>
-<part name="DR_AH" library="jumper" deviceset="J" device="30MM"/>
-<part name="DB_AL" library="jumper" deviceset="J" device="30MM"/>
-<part name="DF_AL" library="jumper" deviceset="J" device="30MM"/>
-<part name="DR_AL" library="jumper" deviceset="J" device="30MM"/>
-<part name="DB_BH" library="jumper" deviceset="J" device="30MM"/>
-<part name="DF_BH" library="jumper" deviceset="J" device="30MM"/>
-<part name="DR_BH" library="jumper" deviceset="J" device="30MM"/>
-<part name="DB_BL" library="jumper" deviceset="J" device="30MM"/>
-<part name="DF_BL" library="jumper" deviceset="J" device="30MM"/>
-<part name="DR_BL" library="jumper" deviceset="J" device="30MM"/>
-<part name="DB_CH" library="jumper" deviceset="J" device="30MM"/>
-<part name="DF_CH" library="jumper" deviceset="J" device="30MM"/>
-<part name="DR_CH" library="jumper" deviceset="J" device="30MM"/>
-<part name="DB_CL" library="jumper" deviceset="J" device="30MM"/>
-<part name="DF_CL" library="jumper" deviceset="J" device="30MM"/>
-<part name="DR_CL" library="jumper" deviceset="J" device="30MM"/>
-<part name="DB_DH" library="jumper" deviceset="J" device="30MM"/>
-<part name="DF_DH" library="jumper" deviceset="J" device="30MM"/>
-<part name="DR_DH" library="jumper" deviceset="J" device="30MM"/>
-<part name="DB_DL" library="jumper" deviceset="J" device="30MM"/>
-<part name="DF_DL" library="jumper" deviceset="J" device="30MM"/>
-<part name="DR_DL" library="jumper" deviceset="J" device="30MM"/>
+<part name="DB_AH" library="jumper" deviceset="J" device="15MM" value="J15MM"/>
+<part name="DF_AH" library="jumper" deviceset="J" device="15MM" value="J15MM"/>
+<part name="DR_AH" library="jumper" deviceset="J" device="15MM" value="J15MM"/>
+<part name="DB_AL" library="jumper" deviceset="J" device="15MM" value="J15MM"/>
+<part name="DF_AL" library="jumper" deviceset="J" device="15MM" value="J15MM"/>
+<part name="DR_AL" library="jumper" deviceset="J" device="15MM" value="J15MM"/>
+<part name="DB_BH" library="jumper" deviceset="J" device="15MM" value="J15MM"/>
+<part name="DF_BH" library="jumper" deviceset="J" device="15MM" value="J15MM"/>
+<part name="DR_BH" library="jumper" deviceset="J" device="15MM" value="J15MM"/>
+<part name="DB_BL" library="jumper" deviceset="J" device="15MM" value="J15MM"/>
+<part name="DF_BL" library="jumper" deviceset="J" device="15MM" value="J15MM"/>
+<part name="DR_BL" library="jumper" deviceset="J" device="15MM" value="J15MM"/>
+<part name="DB_CH" library="jumper" deviceset="J" device="15MM" value="J15MM"/>
+<part name="DF_CH" library="jumper" deviceset="J" device="15MM" value="J15MM"/>
+<part name="DR_CH" library="jumper" deviceset="J" device="15MM" value="J15MM"/>
+<part name="DB_CL" library="jumper" deviceset="J" device="15MM" value="J15MM"/>
+<part name="DF_CL" library="jumper" deviceset="J" device="15MM" value="J15MM"/>
+<part name="DR_CL" library="jumper" deviceset="J" device="15MM" value="J15MM"/>
+<part name="DB_DH" library="jumper" deviceset="J" device="15MM" value="J15MM"/>
+<part name="DF_DH" library="jumper" deviceset="J" device="15MM" value="J15MM"/>
+<part name="DR_DH" library="jumper" deviceset="J" device="15MM" value="J15MM"/>
+<part name="DB_DL" library="jumper" deviceset="J" device="15MM" value="J15MM"/>
+<part name="DF_DL" library="jumper" deviceset="J" device="15MM" value="J15MM"/>
+<part name="DR_DL" library="jumper" deviceset="J" device="15MM" value="J15MM"/>
 <part name="J25" library="jumper" deviceset="J" device="50MM"/>
 <part name="J26" library="jumper" deviceset="J" device="50MM"/>
 <part name="J27" library="jumper" deviceset="J" device="50MM"/>
 <part name="J28" library="jumper" deviceset="J" device="50MM"/>
-<part name="CAP_AH" library="jumper" deviceset="J" device="30MM"/>
-<part name="RES_BASE_AL" library="jumper" deviceset="J" device="30MM"/>
-<part name="CAP_AL" library="jumper" deviceset="J" device="30MM"/>
-<part name="RES_BASE_CH" library="jumper" deviceset="J" device="30MM"/>
-<part name="CAP_CH" library="jumper" deviceset="J" device="30MM"/>
-<part name="RES_BASE_CL" library="jumper" deviceset="J" device="30MM"/>
-<part name="CAP_CL" library="jumper" deviceset="J" device="30MM"/>
-<part name="RES_BASE_BH" library="jumper" deviceset="J" device="30MM"/>
-<part name="CAP_BH" library="jumper" deviceset="J" device="30MM"/>
-<part name="RES_BASE_BL" library="jumper" deviceset="J" device="30MM"/>
-<part name="CAP_BL" library="jumper" deviceset="J" device="30MM"/>
-<part name="RES_BASE_DH" library="jumper" deviceset="J" device="30MM"/>
-<part name="CAP_DH" library="jumper" deviceset="J" device="30MM"/>
-<part name="RES_BASE_DL" library="jumper" deviceset="J" device="30MM"/>
-<part name="CAP_DL" library="jumper" deviceset="J" device="30MM"/>
-<part name="RES_BASE_AH" library="jumper" deviceset="J" device="30MM"/>
+<part name="CAP_AH" library="jumper" deviceset="J" device="15MM" value="J15MM"/>
+<part name="RES_BASE_AL" library="jumper" deviceset="J" device="15MM" value="J15MM"/>
+<part name="CAP_AL" library="jumper" deviceset="J" device="15MM" value="J15MM"/>
+<part name="RES_BASE_CH" library="jumper" deviceset="J" device="15MM" value="J15MM"/>
+<part name="CAP_CH" library="jumper" deviceset="J" device="15MM" value="J15MM"/>
+<part name="RES_BASE_CL" library="jumper" deviceset="J" device="15MM" value="J15MM"/>
+<part name="CAP_CL" library="jumper" deviceset="J" device="15MM" value="J15MM"/>
+<part name="RES_BASE_BH" library="jumper" deviceset="J" device="15MM" value="J15MM"/>
+<part name="CAP_BH" library="jumper" deviceset="J" device="15MM" value="J15MM"/>
+<part name="RES_BASE_BL" library="jumper" deviceset="J" device="15MM" value="J15MM"/>
+<part name="CAP_BL" library="jumper" deviceset="J" device="15MM" value="J15MM"/>
+<part name="RES_BASE_DH" library="jumper" deviceset="J" device="15MM" value="J15MM"/>
+<part name="CAP_DH" library="jumper" deviceset="J" device="15MM" value="J15MM"/>
+<part name="RES_BASE_DL" library="jumper" deviceset="J" device="15MM" value="J15MM"/>
+<part name="CAP_DL" library="jumper" deviceset="J" device="15MM" value="J15MM"/>
+<part name="RES_BASE_AH" library="jumper" deviceset="J" device="15MM" value="J15MM"/>
 <part name="INTERFACE" library="con-lstb" deviceset="MA07-2" device=""/>
 <part name="IC7" library="linear" deviceset="LM358" device="N"/>
 <part name="P+4" library="supply1" deviceset="+5V" device=""/>
 <part name="GND6" library="supply1" deviceset="GND" device=""/>
-<part name="R1" library="resistor" deviceset="R-US_" device="0207/15" value="330 ohm 1w"/>
-<part name="6.8V" library="zener_1n4736A" deviceset="1N4738" device=""/>
-<part name="GND7" library="supply1" deviceset="GND" device=""/>
 <part name="GND8" library="supply1" deviceset="GND" device=""/>
 <part name="SENSE" library="con-wago-500" deviceset="W237-102" device=""/>
@@
 <part name="GND19" library="supply1" deviceset="GND" device=""/>
 <part name="GND20" library="supply1" deviceset="GND" device=""/>
+<part name="P+14" library="supply1" deviceset="+5V" device=""/>
 </parts>
 <sheets>
@@
 <instance part="P+4" gate="1" x="-355.6" y="20.32"/>
 <instance part="GND6" gate="1" x="-314.96" y="7.62"/>
-<instance part="R1" gate="G$1" x="-35.56" y="86.36"/>
-<instance part="6.8V" gate="G$1" x="-20.32" y="81.28" rot="R90"/>
-<instance part="GND7" gate="1" x="-20.32" y="71.12"/>
 <instance part="GND8" gate="1" x="264.16" y="-38.1"/>
 <instance part="SENSE" gate="-1" x="-152.4" y="-10.16"/>
@@
 <instance part="GND19" gate="1" x="386.08" y="-63.5"/>
 <instance part="GND20" gate="1" x="401.32" y="-134.62"/>
+<instance part="P+14" gate="1" x="264.16" y="-10.16"/>
 </instances>
 <busses>
@@
 <wire x1="58.42" y1="15.24" x2="60.96" y2="15.24" width="0.1524" layer="91"/>
 <wire x1="60.96" y1="15.24" x2="60.96" y2="30.48" width="0.1524" layer="91"/>
+</segment>
+<segment>
+<pinref part="IC7" gate="P" pin="V+"/>
+<pinref part="P+14" gate="1" pin="+5V"/>
+<wire x1="264.16" y1="-17.78" x2="264.16" y2="-12.7" width="0.1524" layer="91"/>
 </segment>
 </net>
@@
 <pinref part="SUPPLY2" gate="G$1" pin="VCC"/>
 <wire x1="-48.26" y1="86.36" x2="-48.26" y2="81.28" width="0.1524" layer="91"/>
-<pinref part="R1" gate="G$1" pin="1"/>
-<wire x1="-48.26" y1="86.36" x2="-40.64" y2="86.36" width="0.1524" layer="91"/>
-<junction x="-48.26" y="86.36"/>
 </segment>
 </net>
@@
 <wire x1="233.68" y1="-157.48" x2="223.52" y2="-157.48" width="0.1524" layer="91"/>
 <junction x="223.52" y="-157.48"/>
-</segment>
-<segment>
-<pinref part="GND7" gate="1" pin="GND"/>
-<pinref part="6.8V" gate="G$1" pin="A"/>
-<wire x1="-20.32" y1="73.66" x2="-20.32" y2="78.74" width="0.1524" layer="91"/>
 </segment>
 <segment>
@@
 </segment>
 </net>
-<net name="+6.5V" class="0">
-<segment>
-<pinref part="R1" gate="G$1" pin="2"/>
-<pinref part="6.8V" gate="G$1" pin="C"/>
-<wire x1="-30.48" y1="86.36" x2="-20.32" y2="86.36" width="0.1524" layer="91"/>
-<wire x1="-20.32" y1="86.36" x2="-20.32" y2="83.82" width="0.1524" layer="91"/>
-<wire x1="-20.32" y1="86.36" x2="-20.32" y2="96.52" width="0.1524" layer="91"/>
-<junction x="-20.32" y="86.36"/>
-<junction x="-20.32" y="96.52"/>
-<label x="-17.78" y="96.52" size="1.778" layer="95"/>
-</segment>
-<segment>
-<pinref part="IC7" gate="P" pin="V+"/>
-<junction x="264.16" y="-17.78"/>
-<label x="264.16" y="-15.24" size="1.778" layer="95"/>
-</segment>
-</net>
