File: H_Bridge/h_bridge_board.brd (EAGLE design)
At the start: 100 x 80 mm, 108 parts, among them IC1 74LS08N, IC2 74LS08N, IC3 7805T, IC4 7404N, IC7 LM358N, IC8 LM358N, J1 J50MM, J2 J50MM, J25 J50MM, J26 J50MM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

Commit message: PCB Layoput
Parts:
- moved D8 344.9 mm to (177.8, 17.8), turned to 270 degrees
- moved RES_BASE_DL 323.1 mm to (163.8, 85.1), turned to 90 degrees
- moved OK8 320.5 mm to (168.9, 96.5), turned to 270 degrees
- moved DF_CL 300.1 mm to (142.2, 67.3), turned to 90 degrees
- moved D6 296.8 mm to (177.8, 47.0), turned to 270 degrees
- moved R7 288.2 mm to (147.3, 102.9)
- moved RES_BASE_CL 286.8 mm to (142.2, 85.1), turned to 270 degrees
- moved D7 285.2 mm to (133.3, 17.8), turned to 270 degrees
- moved DB_CL 284.5 mm to (148.6, 67.3), turned to 90 degrees
- moved DB_DH 283.3 mm to (127.0, 67.3), turned to 90 degrees
- moved CAP_DH 280.8 mm to (125.7, 85.1), turned to 90 degrees
- moved CL 276.2 mm to (142.2, 48.3), turned to 90 degrees
- moved DR_CH 273.7 mm to (111.8, 67.3), turned to 90 degrees
- moved OK7 266.8 mm to (124.5, 96.5), turned to 270 degrees
- moved CAP_DL 262.3 mm to (168.9, 85.1), turned to 90 degrees
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Routing:
- net GND: track 0.00 -> 730.3 mm, vias 0 -> 1
- net VCC: track 0.00 -> 493.8 mm
- net +5V: track 0.00 -> 437.5 mm
- net R_SENSE_A_B: track 0.00 -> 349.5 mm
- net R_SENSE_C_D: track 0.00 -> 320.7 mm, vias 0 -> 1
- net IN_D: track 0.00 -> 188.9 mm
- net IN_B: track 0.00 -> 167.7 mm, vias 0 -> 1
- net IN_C: track 0.00 -> 167.0 mm
- net IN_A: track 0.00 -> 150.9 mm
- net OUT_D: track 0.00 -> 148.7 mm
- net OUT_A: track 0.00 -> 136.8 mm
- net OUT_C: track 0.00 -> 134.7 mm
- net SENSE02: track 0.00 -> 131.7 mm
- net ENABLE_A_B: track 0.00 -> 127.9 mm
- net N$13: track 0.00 -> 123.5 mm
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Other:
- board size 100 x 80 mm -> 192.7 x 198.1 mm
